File: bin/sch/ModularDeck/3x3BreakoutBoard/v1.0.0/3x3BreakoutBoard.kicad_sch (KiCad schematic)
At the start: 45 parts

Commit message: First round of bugfixes arising from https://github.com/shanteacontrols/OpenDeck/discussions/173
Parts:
- renumbered KP6 to KP7
Changed lines of the file:
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@@
   (symbol (lib_id "Connector_Generic:Conn_02x04_Top_Bottom") (at 135.89 100.33 0) (unit 1)
     (in_bom yes) (on_board yes) (fields_autoplaced)
-    (property "Reference" "KP6" (id 0) (at 137.16 91.44 0))
+    (property "Reference" "KP7" (id 0) (at 137.16 91.44 0))
     (property "Value" "Conn_02x04_Top_Bottom" (id 1) (at 137.16 93.98 0)
       (effects (font (size 1.27 1.27)) hide)
@@
       (effects (font (size 1.27 1.27)) hide)
     )
-    (property "Description" "To Keypad 6" (id 4) (at 137.16 93.98 0))
+    (property "Description" "To Keypad 7" (id 4) (at 137.16 93.98 0))
     (pin "1")
     (pin "2")
@@
     )
     (path "/a5972cb8-4854-4b37-9fb2-fb1d5ab865eb"
-      (reference "KP6") (unit 1) (value "Conn_02x04_Top_Bottom") (footprint "")
+      (reference "KP7") (unit 1) (value "Conn_02x04_Top_Bottom") (footprint "")
     )
     (path "/4df21a80-b9e5-4aa0-9eba-0b7d570cd0ab"

Commit message: Final changes to 0.0.4 before redoing for 0.1.1
Parts:
- removed D? (x4): ~, symbol Diode:1N4148WT
- added KP8: Conn_02x04_Top_Bottom, symbol Connector_Generic:Conn_02x04_Top_Bottom
- IH? (x2), OH? (x2): symbol Connector_Generic:Conn_02x08_Odd_Even -> Connector_Generic:Conn_02x06_Odd_Even
Connections:
- net BC_6: now also KP8.5 (Pin_5); no longer IH?.13 (Pin_13), IH?.15 (Pin_15)
- net BC_7: now also KP8.7 (Pin_7); no longer IH?.13 (Pin_13), IH?.15 (Pin_15)
- net BR_6: now also KP8.1 (Pin_1)
- net BR_7: now also KP8.3 (Pin_3)
- net LED_COLUMN_6: now also KP8.6 (Pin_6); no longer OH?.14 (Pin_14), OH?.16 (Pin_16)
- net LED_COLUMN_7: now also KP8.8 (Pin_8); no longer OH?.14 (Pin_14), OH?.16 (Pin_16)
- net LED_ROW_0: now also OH?.1 (Pin_1), OH?.1 (Pin_1)
- net LED_ROW_1: now also OH?.3 (Pin_3), OH?.3 (Pin_3); no longer OH?.1 (Pin_1), OH?.1 (Pin_1)
- net LED_ROW_2: now also OH?.5 (Pin_5), OH?.5 (Pin_5); no longer OH?.3 (Pin_3), OH?.3 (Pin_3)
- net LED_ROW_3: now also OH?.7 (Pin_7), OH?.7 (Pin_7); no longer OH?.5 (Pin_5), OH?.5 (Pin_5)
- net LED_ROW_4: now also OH?.9 (Pin_9), OH?.9 (Pin_9); no longer OH?.7 (Pin_7), OH?.7 (Pin_7)
- net LED_ROW_5: now also OH?.11 (Pin_11), OH?.11 (Pin_11); no longer OH?.9 (Pin_9), OH?.9 (Pin_9)
- net LED_ROW_6: now also KP8.2 (Pin_2); no longer OH?.11 (Pin_11), OH?.11 (Pin_11)
- net LED_ROW_7: now also KP8.4 (Pin_4); no longer OH?.13 (Pin_13), OH?.13 (Pin_13)
- removed net LED_ROW_8: OH?.15 (Pin_15), OH?.15 (Pin_15)
Other:
- moved on the sheet: KP7
