File: bin/sch/ModularDeck/3x3BreakoutBoard/v1.0.0/3x3Keypad/3x3Keypad.kicad_sch (KiCad schematic)
At the start: 28 parts

Commit message: Final changes to 0.0.4 before redoing for 0.1.1
Other:
- moved on the sheet: BRK?, D?, KSW?
