File: bin/sch/MOOD/v0.1.1/Motherboard/DMX.kicad_sch (KiCad schematic)
At the start: 12 parts, among them J4 XLR3, U11 6N137, U12 MAX485, U13 B0505S-1WR3

Commit message: Finished version 0.1.1 of motherboard
Parts:
- C?: renamed from C13; value 4.7u -> 10u
- U?: renamed from U13; value B0505S-1WR3 -> RFM-0505
- renumbered C33 to C?, C12 to C?, C34 to C?, C11 to C?, J4 to J?, R21 to R?, R24 to R?, R22 to R?, U11 to U?, U12 to U?
Changed lines of the file:
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@@
   (symbol (lib_id "Connector:XLR3") (at 215.9 85.09 0) (mirror y) (unit 1)
     (in_bom yes) (on_board yes) (fields_autoplaced)
-    (property "Reference" "J4" (id 0) (at 215.9 74.93 0))
+    (property "Reference" "J?" (id 0) (at 215.9 74.93 0))
     (property "Value" "XLR3" (id 1) (at 215.9 77.47 0))
     (property "Footprint" "igor_footprint_lib:TRAPC3MX" (id 2) (at 215.9 85.09 0)
@@
   (symbol (lib_id "power:GND1") (at 223.52 85.09 90) (unit 1)
     (in_bom yes) (on_board yes)
-    (property "Reference" "#PWR0162" (id 0) (at 229.87 85.09 0)
+    (property "Reference" "#PWR?" (id 0) (at 229.87 85.09 0)
       (effects (font (size 1.27 1.27)) hide)
     )
@@
   (symbol (lib_id "power:GND1") (at 118.11 77.47 270) (mirror x) (unit 1)
     (in_bom yes) (on_board yes)
-    (property "Reference" "#PWR0153" (id 0) (at 111.76 77.47 0)
+    (property "Reference" "#PWR?" (id 0) (at 111.76 77.47 0)
       (effects (font (size 1.27 1.27)) hide)
     )
@@
   (symbol (lib_id "igor_lib:6N137") (at 130.81 92.71 0) (unit 1)
     (in_bom yes) (on_board yes)
-    (property "Reference" "U11" (id 0) (at 137.16 71.12 0))
+    (property "Reference" "U?" (id 0) (at 137.16 71.12 0))
     (property "Value" "6N137" (id 1) (at 137.16 73.66 0))
     (property "Footprint" "Package_SO:SSO-8_6.7x9.8mm_P2.54mm_Clearance8mm" (id 2) (at 137.16 97.79 0)
@@
   (symbol (lib_id "power:GND1") (at 87.63 86.36 90) (mirror x) (unit 1)
     (in_bom yes) (on_board yes)
-    (property "Reference" "#PWR0156" (id 0) (at 93.98 86.36 0)
+    (property "Reference" "#PWR?" (id 0) (at 93.98 86.36 0)
       (effects (font (size 1.27 1.27)) hide)
     )
@@
   (symbol (lib_id "power:+3.3V") (at 125.73 85.09 90) (unit 1)
     (in_bom yes) (on_board yes)
-    (property "Reference" "#PWR0151" (id 0) (at 129.54 85.09 0)
+    (property "Reference" "#PWR?" (id 0) (at 129.54 85.09 0)
       (effects (font (size 1.27 1.27)) hide)
     )
@@
   (symbol (lib_id "power:+5VD") (at 87.63 81.28 270) (unit 1)
     (in_bom yes) (on_board yes)
-    (property "Reference" "#PWR0158" (id 0) (at 83.82 81.28 0)
+    (property "Reference" "#PWR?" (id 0) (at 83.82 81.28 0)
       (effects (font (size 1.27 1.27)) hide)
     )
@@
   (symbol (lib_id "Device:C") (at 58.42 81.28 90) (unit 1)
     (in_bom yes) (on_board yes)
-    (property "Reference" "C13" (id 0) (at 58.42 74.93 90))
-    (property "Value" "4.7u" (id 1) (at 58.42 77.47 90))
+    (property "Reference" "C?" (id 0) (at 58.42 74.93 90))
+    (property "Value" "10u" (id 1) (at 58.42 77.47 90))
     (property "Footprint" "Capacitor_SMD:C_0402_1005Metric" (id 2) (at 62.23 80.3148 0)
       (effects (font (size 1.27 1.27)) hide)
@@
   (symbol (lib_id "igor_lib:MAX485") (at 173.99 87.63 0) (unit 1)
     (in_bom yes) (on_board yes) (fields_autoplaced)
-    (property "Reference" "U12" (id 0) (at 181.61 62.23 0))
+    (property "Reference" "U?" (id 0) (at 181.61 62.23 0))
     (property "Value" "MAX485" (id 1) (at 181.61 64.77 0))
     (property "Footprint" "Package_SO:SO-8_3.9x4.9mm_P1.27mm" (id 2) (at 173.99 92.71 0)
@@
   (symbol (lib_id "power:GND1") (at 87.63 73.66 0) (mirror x) (unit 1)
     (in_bom yes) (on_board yes)
-    (property "Reference" "#PWR014" (id 0) (at 87.63 67.31 0)
+    (property "Reference" "#PWR?" (id 0) (at 87.63 67.31 0)
       (effects (font (size 1.27 1.27)) hide)
     )
@@
   (symbol (lib_id "Device:C") (at 58.42 69.85 90) (unit 1)
     (in_bom yes) (on_board yes)
-    (property "Reference" "C33" (id 0) (at 58.42 63.5 90))
+    (property "Reference" "C?" (id 0) (at 58.42 63.5 90))
     (property "Value" "4.7u" (id 1) (at 58.42 66.04 90))
     (property "Footprint" "Capacitor_SMD:C_0402_1005Metric" (id 2) (at 62.23 68.8848 0)
@@
   (symbol (lib_id "power:GND") (at 49.53 81.28 270) (unit 1)
     (in_bom yes) (on_board yes)
-    (property "Reference" "#PWR0159" (id 0) (at 43.18 81.28 0)
+    (property "Reference" "#PWR?" (id 0) (at 43.18 81.28 0)
       (effects (font (size 1.27 1.27)) hide)
     )
@@
   (symbol (lib_id "power:+5V") (at 62.23 66.04 0) (unit 1)
     (in_bom yes) (on_board yes)
-    (property "Reference" "#PWR0160" (id 0) (at 62.23 69.85 0)
+    (property "Reference" "#PWR?" (id 0) (at 62.23 69.85 0)
       (effects (font (size 1.27 1.27)) hide)
     )
@@
   (symbol (lib_id "Device:C") (at 165.1 69.85 90) (unit 1)
     (in_bom yes) (on_board yes)
-    (property "Reference" "C12" (id 0) (at 165.1 62.23 90))
+    (property "Reference" "C?" (id 0) (at 165.1 62.23 90))
     (property "Value" "100n" (id 1) (at 165.1 64.77 90))
     (property "Footprint" "Capacitor_SMD:C_0402_1005Metric" (id 2) (at 168.91 68.8848 0)
@@
   (symbol (lib_id "power:+5VD") (at 168.91 80.01 90) (unit 1)
     (in_bom yes) (on_board yes)
-    (property "Reference" "#PWR0154" (id 0) (at 172.72 80.01 0)
+    (property "Reference" "#PWR?" (id 0) (at 172.72 80.01 0)
       (effects (font (size 1.27 1.27)) hide)
     )
@@
   (symbol (lib_id "power:+5VD") (at 152.4 77.47 0) (unit 1)
     (in_bom yes) (on_board yes)
-    (property "Reference" "#PWR0150" (id 0) (at 152.4 81.28 0)
+    (property "Reference" "#PWR?" (id 0) (at 152.4 81.28 0)
       (effects (font (size 1.27 1.27)) hide)
     )
@@
   (symbol (lib_id "Device:R") (at 121.92 90.17 90) (unit 1)
     (in_bom yes) (on_board yes)
-    (property "Reference" "R21" (id 0) (at 121.92 87.63 90))
+    (property "Reference" "R?" (id 0) (at 121.92 87.63 90))
     (property "Value" "470" (id 1) (at 121.92 90.17 90))
     (property "Footprint" "Resistor_SMD:R_0402_1005Metric" (id 2) (at 121.92 91.948 90)
@@
   (symbol (lib_id "Device:R") (at 198.12 81.28 0) (unit 1)
     (in_bom yes) (on_board yes)
-    (property "Reference" "R24" (id 0) (at 200.66 81.28 90))
+    (property "Reference" "R?" (id 0) (at 200.66 81.28 90))
     (property "Value" "133" (id 1) (at 198.12 81.28 90))
     (property "Footprint" "Resistor_SMD:R_0402_1005Metric" (id 2) (at 196.342 81.28 90)
@@
   (symbol (lib_id "Device:R") (at 152.4 81.28 0) (unit 1)
     (in_bom yes) (on_board yes)
-    (property "Reference" "R22" (id 0) (at 154.94 81.28 90))
+    (property "Reference" "R?" (id 0) (at 154.94 81.28 90))
     (property "Value" "4.7k" (id 1) (at 152.4 81.28 90))
     (property "Footprint" "Resistor_SMD:R_0402_1005Metric" (id 2) (at 150.622 81.28 90)
@@
   (symbol (lib_id "power:GND1") (at 161.29 69.85 270) (unit 1)
     (in_bom yes) (on_board yes)
-    (property "Reference" "#PWR0157" (id 0) (at 154.94 69.85 0)
+    (property "Reference" "#PWR?" (id 0) (at 154.94 69.85 0)
       (effects (font (size 1.27 1.27)) hide)
     )
@@
   (symbol (lib_id "power:GND") (at 49.53 69.85 270) (unit 1)
     (in_bom yes) (on_board yes)
-    (property "Reference" "#PWR0155" (id 0) (at 43.18 69.85 0)
+    (property "Reference" "#PWR?" (id 0) (at 43.18 69.85 0)
       (effects (font (size 1.27 1.27)) hide)
     )
@@
   (symbol (lib_id "Device:C") (at 87.63 77.47 0) (unit 1)
     (in_bom yes) (on_board yes)
-    (property "Reference" "C34" (id 0) (at 91.44 72.39 0))
+    (property "Reference" "C?" (id 0) (at 91.44 72.39 0))
     (property "Value" "10u" (id 1) (at 91.44 74.93 0))
     (property "Footprint" "Capacitor_SMD:C_0402_1005Metric" (id 2) (at 88.5952 81.28 0)
@@
   (symbol (lib_id "igor_lib:RFM-0505") (at 67.31 88.9 0) (unit 1)
     (in_bom yes) (on_board yes) (fields_autoplaced)
-    (property "Reference" "U13" (id 0) (at 74.93 73.66 0))
-    (property "Value" "B0505S-1WR3" (id 1) (at 74.93 76.2 0))
+    (property "Reference" "U?" (id 0) (at 74.93 73.66 0))
+    (property "Value" "RFM-0505" (id 1) (at 74.93 76.2 0))
     (property "Footprint" "igor_footprint_lib:RFM-0505" (id 2) (at 67.31 88.9 0)
       (effects (font (size 1.27 1.27)) hide)
@@
   (symbol (lib_id "power:+5VD") (at 125.73 72.39 0) (unit 1)
     (in_bom yes) (on_board yes)
-    (property "Reference" "#PWR022" (id 0) (at 125.73 76.2 0)
+    (property "Reference" "#PWR?" (id 0) (at 125.73 76.2 0)
       (effects (font (size 1.27 1.27)) hide)
     )
@@
   (symbol (lib_id "power:+5VD") (at 168.91 64.77 0) (unit 1)
     (in_bom yes) (on_board yes)
-    (property "Reference" "#PWR0149" (id 0) (at 168.91 68.58 0)
+    (property "Reference" "#PWR?" (id 0) (at 168.91 68.58 0)
       (effects (font (size 1.27 1.27)) hide)
     )
@@
   (symbol (lib_id "Device:C") (at 121.92 77.47 90) (unit 1)
     (in_bom yes) (on_board yes)
-    (property "Reference" "C11" (id 0) (at 121.92 69.85 90))
+    (property "Reference" "C?" (id 0) (at 121.92 69.85 90))
     (property "Value" "100n" (id 1) (at 121.92 72.39 90))
     (property "Footprint" "Capacitor_SMD:C_0402_1005Metric" (id 2) (at 125.73 76.5048 0)
@@
   (symbol (lib_id "power:GND") (at 49.53 86.36 270) (mirror x) (unit 1)
     (in_bom yes) (on_board yes)
-    (property "Reference" "#PWR0161" (id 0) (at 43.18 86.36 0)
-      (effects (font (size 1.27 1.27)) hide)
-    )
+    (property "Reference" "#PWR?" (id 0) (at 43.18 86.36 0)
+      (effects (font (size 1.27 1.27)) hide)
+    )
