File: bin/sch/MOOD/v0.1.1/Motherboard/DIN_Serial.kicad_sch (KiCad schematic)
At the start: 28 parts, among them J2 DIN-5, U10 TLP2362

Commit message: -	Made a bunch of changes -	Added KeyboardCard
Parts:
- C46, C47: renamed from C?; footprint (none) -> Capacitor_SMD:C_0402_1005Metric
- gave numbers to parts that had none: 20

Commit message: -	Hopefully finished schematics -	Started desining PCB for motherboard
Parts:
- removed D13, D14: Green, LED_SMD:LED_0805_2012Metric, symbol Device:LED
- removed D15: Blue, LED_SMD:LED_0805_2012Metric, symbol Device:LED
- removed R44, R45: 680, Resistor_SMD:R_0402_1005Metric, symbol Device:R
- removed R46: 1k, Resistor_SMD:R_0402_1005Metric, symbol Device:R
Changed lines of the file:
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@@
-    (effects (font (size 1.27 1.27)) (justify left))
-  )
-  (hierarchical_label "DMX_TRAFFIC_OUT" (shape input) (at 196.85 165.1 90)
     (effects (font (size 1.27 1.27)) (justify left))
   )
   (hierarchical_label "MIDI_TX" (shape input) (at 254 199.39 180)
     (effects (font (size 1.27 1.27)) (justify right))
-  )
-  (hierarchical_label "MIDI_TRAFFIC_IN" (shape input) (at 209.55 165.1 90)
-    (effects (font (size 1.27 1.27)) (justify left))
-  )
-  (hierarchical_label "MIDI_TRAFFIC_OUT" (shape input) (at 220.98 165.1 90)
-    (effects (font (size 1.27 1.27)) (justify left))
   )
   (symbol (lib_id "MOOD_Library:+5V-SerialOut") (at 369.57 147.32 270) (unit 1)
@@
     (pin "1")
   )
-  (symbol (lib_id "power:GND") (at 220.98 180.34 0) (unit 1)
-    (in_bom yes) (on_board yes)
-    (property "Reference" "#PWR0187" (id 0) (at 220.98 186.69 0)
-      (effects (font (size 1.27 1.27)) hide)
-    )
-    (property "Value" "GND" (id 1) (at 218.44 184.15 0)
-      (effects (font (size 1.27 1.27)) (justify left))
-    )
-    (property "Footprint" "" (id 2) (at 220.98 180.34 0)
-      (effects (font (size 1.27 1.27)) hide)
-    )
-    (property "Datasheet" "" (id 3) (at 220.98 180.34 0)
-      (effects (font (size 1.27 1.27)) hide)
-    )
-    (pin "1")
-  )
   (symbol (lib_id "Device:R") (at 334.01 77.47 0) (unit 1)
     (in_bom yes) (on_board yes)
@@
     (pin "1")
   )
-  (symbol (lib_id "Device:R") (at 196.85 168.91 0) (unit 1)
-    (in_bom yes) (on_board yes)
-    (property "Reference" "R44" (id 0) (at 199.39 168.91 90))
-    (property "Value" "680" (id 1) (at 196.85 168.91 90))
-    (property "Footprint" "Resistor_SMD:R_0402_1005Metric" (id 2) (at 195.072 168.91 90)
-      (effects (font (size 1.27 1.27)) hide)
-    )
-    (property "Datasheet" "~" (id 3) (at 196.85 168.91 0)
-      (effects (font (size 1.27 1.27)) hide)
-    )
-    (property "LCSC" "C25130" (id 4) (at 196.85 168.91 0)
-      (effects (font (size 1.27 1.27)) hide)
-    )
-    (pin "1")
-    (pin "2")
-  )
   (symbol (lib_id "power:GND1") (at 369.57 139.7 0) (mirror x) (unit 1)
     (in_bom yes) (on_board yes)
@@
     )
     (property "LCSC" "C25105" (id 4) (at 375.92 219.71 0)
-      (effects (font (size 1.27 1.27)) hide)
-    )
-    (pin "1")
-    (pin "2")
-  )
-  (symbol (lib_id "Device:R") (at 209.55 168.91 0) (unit 1)
-    (in_bom yes) (on_board yes)
-    (property "Reference" "R45" (id 0) (at 212.09 168.91 90))
-    (property "Value" "680" (id 1) (at 209.55 168.91 90))
-    (property "Footprint" "Resistor_SMD:R_0402_1005Metric" (id 2) (at 207.772 168.91 90)
-      (effects (font (size 1.27 1.27)) hide)
-    )
-    (property "Datasheet" "~" (id 3) (at 209.55 168.91 0)
-      (effects (font (size 1.27 1.27)) hide)
-    )
-    (property "LCSC" "C25130" (id 4) (at 209.55 168.91 0)
-      (effects (font (size 1.27 1.27)) hide)
-    )
-    (pin "1")
-    (pin "2")
-  )
-  (symbol (lib_id "power:GND") (at 209.55 180.34 0) (unit 1)
-    (in_bom yes) (on_board yes)
-    (property "Reference" "#PWR0186" (id 0) (at 209.55 186.69 0)
-      (effects (font (size 1.27 1.27)) hide)
-    )
-    (property "Value" "GND" (id 1) (at 207.01 184.15 0)
-      (effects (font (size 1.27 1.27)) (justify left))
-    )
-    (property "Footprint" "" (id 2) (at 209.55 180.34 0)
-      (effects (font (size 1.27 1.27)) hide)
-    )
-    (property "Datasheet" "" (id 3) (at 209.55 180.34 0)
-      (effects (font (size 1.27 1.27)) hide)
-    )
-    (pin "1")
-  )
-  (symbol (lib_id "Device:R") (at 220.98 168.91 0) (unit 1)
-    (in_bom yes) (on_board yes)
-    (property "Reference" "R46" (id 0) (at 223.52 168.91 90))
-    (property "Value" "1k" (id 1) (at 220.98 168.91 90))
-    (property "Footprint" "Resistor_SMD:R_0402_1005Metric" (id 2) (at 219.202 168.91 90)
-      (effects (font (size 1.27 1.27)) hide)
-    )
-    (property "Datasheet" "~" (id 3) (at 220.98 168.91 0)
-      (effects (font (size 1.27 1.27)) hide)
-    )
-    (property "LCSC" "C11702" (id 4) (at 220.98 168.91 0)
       (effects (font (size 1.27 1.27)) hide)
     )
@@
     (pin "1")
   )
-  (symbol (lib_id "Device:LED") (at 196.85 176.53 90) (unit 1)
-    (in_bom yes) (on_board yes)
-    (property "Reference" "D13" (id 0) (at 199.39 176.53 0))
-    (property "Value" "Green" (id 1) (at 201.93 178.1175 0)
-      (effects (font (size 1.27 1.27)) hide)
-    )
-    (property "Footprint" "LED_SMD:LED_0805_2012Metric" (id 2) (at 196.85 176.53 0)
-      (effects (font (size 1.27 1.27)) hide)
-    )
-    (property "Datasheet" "~" (id 3) (at 196.85 176.53 0)
-      (effects (font (size 1.27 1.27)) hide)
-    )
-    (property "LCSC" "C142303" (id 4) (at 196.85 176.53 0)
-      (effects (font (size 1.27 1.27)) hide)
-    )
-    (pin "1")
-    (pin "2")
-  )
   (symbol (lib_id "power:GND") (at 289.56 220.98 0) (unit 1)
     (in_bom yes) (on_board yes) (fields_autoplaced)
@@
     (pin "4")
   )
-  (symbol (lib_id "power:GND") (at 196.85 180.34 0) (unit 1)
-    (in_bom yes) (on_board yes)
-    (property "Reference" "#PWR0185" (id 0) (at 196.85 186.69 0)
-      (effects (font (size 1.27 1.27)) hide)
-    )
-    (property "Value" "GND" (id 1) (at 194.31 184.15 0)
-      (effects (font (size 1.27 1.27)) (justify left))
-    )
-    (property "Footprint" "" (id 2) (at 196.85 180.34 0)
-      (effects (font (size 1.27 1.27)) hide)
-    )
-    (property "Datasheet" "" (id 3) (at 196.85 180.34 0)
-      (effects (font (size 1.27 1.27)) hide)
-    )
-    (pin "1")
-  )
   (symbol (lib_name "DIN-5_1") (lib_id "Connector:DIN-5") (at 363.22 222.25 0) (unit 1)
     (in_bom yes) (on_board yes)
@@
     (pin "1")
   )
-  (symbol (lib_id "Device:LED") (at 209.55 176.53 90) (unit 1)
-    (in_bom yes) (on_board yes)
-    (property "Reference" "D14" (id 0) (at 212.09 176.53 0))
-    (property "Value" "Green" (id 1) (at 214.63 178.1175 0)
-      (effects (font (size 1.27 1.27)) hide)
-    )
-    (property "Footprint" "LED_SMD:LED_0805_2012Metric" (id 2) (at 209.55 176.53 0)
-      (effects (font (size 1.27 1.27)) hide)
-    )
-    (property "Datasheet" "~" (id 3) (at 209.55 176.53 0)
-      (effects (font (size 1.27 1.27)) hide)
-    )
-    (property "LCSC" "C142303" (id 4) (at 209.55 176.53 0)
-      (effects (font (size 1.27 1.27)) hide)
-    )
-    (pin "1")
-    (pin "2")
-  )
   (symbol (lib_id "Device:C") (at 283.21 180.34 90) (unit 1)
     (in_bom yes) (on_board yes)
@@
     (pin "1")
   )
-  (symbol (lib_id "Device:LED") (at 220.98 176.53 90) (unit 1)
-    (in_bom yes) (on_board yes)
-    (property "Reference" "D15" (id 0) (at 223.52 176.53 0))
-    (property "Value" "Blue" (id 1) (at 226.06 178.1175 0)
-      (effects (font (size 1.27 1.27)) hide)
-    )
-    (property "Footprint" "LED_SMD:LED_0805_2012Metric" (id 2) (at 220.98 176.53 0)
-      (effects (font (size 1.27 1.27)) hide)
-    )
-    (property "Datasheet" "~" (id 3) (at 220.98 176.53 0)
-      (effects (font (size 1.27 1.27)) hide)
-    )
-    (property "LCSC" "C84259" (id 4) (at 220.98 176.53 0)
-      (effects (font (size 1.27 1.27)) hide)
-    )
-    (pin "1")
-    (pin "2")
-  )
   (symbol (lib_id "MOOD_Library:+3.3V-Switched") (at 307.34 68.58 0) (unit 1)

Commit message: Finalised schematic and PCB for MOOD Motherboard
Parts:
- R48: footprint (none) -> Resistor_SMD:R_0402_1005Metric
- U13: footprint (none) -> Package_SO:SOIC-8_3.9x4.9mm_P1.27mm
Changed lines of the file:
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@@
       (effects (font (size 1.27 1.27)) (justify left))
     )
-    (property "Footprint" "" (id 2) (at 345.44 207.01 0)
+    (property "Footprint" "Package_SO:SOIC-8_3.9x4.9mm_P1.27mm" (id 2) (at 345.44 207.01 0)
       (effects (font (size 1.27 1.27)) hide)
     )
@@
       (effects (font (size 1.27 1.27)) (justify left))
     )
-    (property "Footprint" "" (id 2) (at 271.78 187.452 90)
+    (property "Footprint" "Resistor_SMD:R_0402_1005Metric" (id 2) (at 271.78 187.452 90)
       (effects (font (size 1.27 1.27)) hide)
     )
@@
   )
   (symbol (lib_id "power:GND") (at 284.48 160.02 270) (unit 1)
-    (in_bom yes) (on_board yes)
+    (in_bom yes) (on_board yes) (fields_autoplaced)
     (property "Reference" "#PWR0180" (id 0) (at 278.13 160.02 0)
       (effects (font (size 1.27 1.27)) hide)
     )
-    (property "Value" "~" (id 1) (at 280.67 157.48 90)
-      (effects (font (size 1.27 1.27)) (justify left))
+    (property "Value" "GND" (id 1) (at 280.67 160.0199 90)
+      (effects (font (size 1.27 1.27)) (justify right))
     )
     (property "Footprint" "" (id 2) (at 284.48 160.02 0)
