File: bin/sch/MOOD/v0.1.1/Motherboard/Ethernet_to_SPI.kicad_sch (KiCad schematic)
At the start: 11 parts

Commit message: -	Made a bunch of changes -	Added KeyboardCard
Parts:
- C52, C53: renamed from C?; footprint (none) -> Capacitor_SMD:C_0402_1005Metric
- gave numbers to parts that had none: 9
Connections:
- net +3.3V renamed +3.3V-Supply

Commit message: Finalised schematic and PCB for MOOD Motherboard
Parts:
- R52, R53, R54, R55, R56: footprint (none) -> Resistor_SMD:R_0402_1005Metric
Changed lines of the file:
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@@
       (effects (font (size 1.27 1.27)) (justify left))
     )
-    (property "Footprint" "" (id 2) (at 145.542 81.28 90)
+    (property "Footprint" "Resistor_SMD:R_0402_1005Metric" (id 2) (at 145.542 81.28 90)
       (effects (font (size 1.27 1.27)) hide)
     )
@@
       (effects (font (size 1.27 1.27)) hide)
     )
-    (property "Datasheet" "http://wizwiki.net/wiki/lib/exe/fetch.php/products:w5500:w5500_ds_v109e.pdf" (id 3) (at 105.41 41.91 0)
+    (property "Datasheet" "https://docs.wiznet.io/img/products/w5500/W5500_ds_v110e.pdf" (id 3) (at 105.41 41.91 0)
       (effects (font (size 1.27 1.27)) hide)
     )
@@
     )
     (property "Value" "4.7k" (id 1) (at 140.97 44.45 90))
-    (property "Footprint" "" (id 2) (at 139.192 44.45 90)
+    (property "Footprint" "Resistor_SMD:R_0402_1005Metric" (id 2) (at 139.192 44.45 90)
       (effects (font (size 1.27 1.27)) hide)
     )
@@
       (effects (font (size 1.27 1.27)) (justify left))
     )
-    (property "Footprint" "" (id 2) (at 153.162 81.28 90)
+    (property "Footprint" "Resistor_SMD:R_0402_1005Metric" (id 2) (at 153.162 81.28 90)
       (effects (font (size 1.27 1.27)) hide)
     )
@@
       (effects (font (size 1.27 1.27)) (justify left))
     )
-    (property "Footprint" "" (id 2) (at 56.642 92.71 90)
+    (property "Footprint" "Resistor_SMD:R_0402_1005Metric" (id 2) (at 56.642 92.71 90)
       (effects (font (size 1.27 1.27)) hide)
     )
@@
     )
     (property "Value" "4.7k" (id 1) (at 123.19 34.29 90))
-    (property "Footprint" "" (id 2) (at 121.412 34.29 90)
-      (effects (font (size 1.27 1.27)) hide)
-    )
+    (property "Footprint" "Resistor_SMD:R_0402_1005Metric" (id 2) (at 121.412 34.29 90)
+      (effects (font (size 1.27 1.27)) hide)
+    )
