File: bin/sch/MOOD/v0.1.1/Motherboard/MOOD-Motherboard-r0.1.1.kicad_pcb (KiCad board)
At the start: 2 copper layers, 181 x 97 mm, 262 parts, among them J1 DIN-5, J10 Conn_01x03, J11 Conn_01x02, J2 DIN-5, J3 Conn_01x04, J5 Conn_01x02, J6 Conn_01x04, J7 Conn_01x04, J8 Conn_01x04, J9 TYPE-C-31-M-12, U1 74HC4067, U10 TLP2362, U11 74HCT125, U12 74HCT125, U14 SPX3819M5, U15 W25Q128JVS, U16 SPX3819M5, U17 RP2040, U18 4051, U2 74HC4067, U3 74HC4067, U4 74HC165, U5 74HC138, U6 MAX7219, U7 74HC4067, U8 74HC165, U9 74HCT125, Y1 12MHz

Commit message: -	Hopefully finished schematics -	Started desining PCB for motherboard
Parts:
- removed AH1, AH2, AH3, AH4, AH5, AH6, AH7, AH8: 3x08, igor_footprint_lib:3x08
- removed C1, C11, C12, C2, C3, C35, C4, C5, C6, C7, C8, C9: 100n, Capacitor_SMD:C_0402_1005Metric
- removed C14: 1u, Capacitor_SMD:C_0402_1005Metric
- removed D1, D10, D100, D101, D102, D103, D104, D105, D106, D107, D108, D109, D11, D110, D111, D112, D113, D114, D115, D116, D117, D118, D119, D12, D120, D121, D122, D123, D124, D125, D126, D127, D128, D129, D13, D14, D15, D16, D17, D18, D19, D2, D20, D21, D22, D23, D24, D25, D26, D27, D28, D29, D3, D30, D31, D32, D34, D35, D36, D37, D38, D39, D4, D40, D41, D42, D43, D44, D45, D46, D47, D48, D49, D5, D50, D51, D52, D53, D54, D55, D56, D57, D58, D59, D6, D60, D61, D62, D63, D64, D65, D66, D67, D68, D69, D7, D70, D71, D72, D73, D74, D75, D76, D77, D78, D79, D8, D80, D81, D82, D83, D84, D85, D86, D87, D88, D89, D9, D90, D91, D92, D93, D94, D95, D96, D97, D98, D99: 1N4148WT, Diode_SMD:D_SOD-523
- removed D131: Green, LED_SMD:LED_0805_2012Metric
- removed D132: Blue, LED_SMD:LED_0805_2012Metric
- removed IH1, IH10, IH11, IH12, IH13, IH14, IH15, IH16, IH2, IH3, IH4, IH5, IH6, IH7, IH8, IH9, OH1, OH2, OH3, OH4, OH5, OH6, OH7, OH8: Conn_02x08_Top_Bottom, Connector_PinHeader_2.54mm:PinHeader_2x08_P2.54mm_Vertical
- removed J3: Conn_01x04, Connector_JST:JST_XH_B4B-XH-A_1x04_P2.50mm_Vertical
- removed the J6 at (208.5, 73.4)
- removed R1, R10, R11, R12, R13, R14, R15, R16, R2, R3, R4, R5, R6, R7, R8, R9: 4.7k, Resistor_SMD:R_0402_1005Metric
- removed R25: 680, Resistor_SMD:R_0402_1005Metric
- removed R26: 10k, Resistor_SMD:R_0402_1005Metric
- removed R27: 1k, Resistor_SMD:R_0402_1005Metric
- removed U1, U2, U3, U7: 74HC4067, Package_SO:SOIC-24W_7.5x15.4mm_P1.27mm
- removed U11, U12: 74HCT125, Package_SO:TSSOP-14_4.4x5mm_P0.65mm
- removed U18: 4051, Package_SO:SOIC-16_3.9x9.9mm_P1.27mm
- removed U4, U8: 74HC165, Package_SO:SO-16_3.9x9.9mm_P1.27mm
- removed U5: 74HC138, Package_SO:SO-16_3.9x9.9mm_P1.27mm
- removed U6: MAX7219, Package_SO:SOIC-24W_7.5x15.4mm_P1.27mm
- removed the U9 at (158.2, 87.5)
- added C50: 10u, Capacitor_SMD:C_0402_1005Metric, F.Cu at (181.3, 40.4)
- added J12: XLR3, igor_footprint_lib:TRAPC3MX, F.Cu at (176.2, 31.1)
- added U13: MAX485, Package_SO:SO-8_3.9x4.9mm_P1.27mm, F.Cu at (180.7, 48.5)
- U14: value SPX3819M5 -> RFM-0505; footprint Package_TO_SOT_SMD:SOT-23-5 -> igor_footprint_lib:RFM-0505
- moved U14 83.2 mm to (178.3, 40.3)
- renumbered C31 to C42, C15 to C44, C16 to C45, J8 to J6, J9 to J8, J1 to J9, R23 to R2300, R29 to R40, R30 to R41, R17 to R50, R18 to R51, U16 to U9
Connections:
- C10 pad 2: +3V3 -> +3.3V-Switched
- C17 pad 1: +3V3 -> +3.3V-Switched
- C18 pad 1: +3V3 -> +3.3V-Switched
- C19 pad 1: +3V3 -> +3.3V-Switched
- C20 pad 1: +3V3 -> +3.3V-Switched
- C21 pad 1: +3V3 -> +3.3V-Switched
- C22 pad 1: +3V3 -> +3.3V-Switched
- C24 pad 1: +3V3 -> +3.3V-Switched
- C26 pad 1: +3V3 -> +3.3V-Switched
- C30 pad 1: +3V3 -> +3.3V-Switched
- C32 pad 1: +3V3 -> +3.3V-Switched
- J2 pad 6: unconnected-(J2-Pad6) -> (no net)
- J2 pad 7: unconnected-(J2-Pad7) -> (no net)
- J2 pad 8: unconnected-(J2-Pad8) -> (no net)
- J2 pad 9: unconnected-(J2-Pad9) -> (no net)
- R20 pad 1: +3V3 -> +3.3V-Switched
- R34 pad 1: +3V3 -> +3.3V-Switched
- R35 pad 1: +3V3 -> +3.3V-Switched
- U10 pad 6: +3V3 -> +3.3V-Switched
- U14 pad 1: +5V -> GND
- U14 pad 2: GND -> +5V
- U14 pad 3: +5V -> (no net)
- U14 pad 4: unconnected-(U14-Pad4) -> (no net)
- U17 pad 1: +3V3 -> +3.3V-Switched
- U17 pad 10: +3V3 -> +3.3V-Switched
- U17 pad 11: /SR_IN_DATA -> /SPI1_RX
- U17 pad 12: /DEC_DI_A2 -> /SPI1_CSn
- U17 pad 13: /DEC_DI_A1 -> /SPI1_SCK
- U17 pad 14: /DEC_DI_A0 -> /SPI1_TX
- U17 pad 15: unconnected-(U17-Pad15) -> /ETH_RSTn
- U17 pad 16: unconnected-(U17-Pad16) -> /ETH_INTn
- U17 pad 17: /MAX7219_DIN -> /PSW_KILL
- U17 pad 18: /MAX7219_LOAD -> /PSW_INT
- U17 pad 22: +3V3 -> +3.3V-Switched
- U17 pad 27: unconnected-(U17-Pad27) -> /SPI0_RX
- U17 pad 28: unconnected-(U17-Pad28) -> /SPI0_CS0
- U17 pad 29: /BTLDR -> /SPI0_SCK
- U17 pad 30: /TRAFFIC_OUT -> /SPI0_TX
- U17 pad 31: /TRAFFIC_IN -> /SPI0_CS1
- U17 pad 32: unconnected-(U17-Pad32) -> /SPI0_CS2
- U17 pad 33: +3V3 -> +3.3V-Switched
- U17 pad 34: /MUX_S3 -> /SPI0_CS3
- U17 pad 35: /MUX_S2 -> /SPI0_CS4
- U17 pad 36: /MUX_S0 -> /SPI0_CS5
- U17 pad 37: /MUX_S1 -> /CLOCK_SUB
- U17 pad 38: /MUX_SEL0 -> unconnected-(U17-Pad38)
- U17 pad 39: /MUX_SEL1 -> unconnected-(U17-Pad39)
- U17 pad 4: /SDA -> /BTLDR
- U17 pad 40: /MUX_COMMON -> unconnected-(U17-Pad40)
- U17 pad 42: +3V3 -> +3.3V-Switched
- U17 pad 43: +3V3 -> +3.3V-Switched
- U17 pad 44: +3V3 -> +3.3V-Switched
- U17 pad 48: +3V3 -> +3.3V-Switched
- U17 pad 49: +3V3 -> +3.3V-Switched
- U17 pad 5: /SCL -> unconnected-(U17-Pad5)
- U17 pad 6: /TSCREEN_TX -> /DMI_TX
- U17 pad 7: /TSCREEN_RX -> unconnected-(U17-Pad7)
- U17 pad 8: /SR_IN_LATCH -> unconnected-(U17-Pad8)
- U17 pad 9: /SPI_CLK -> unconnected-(U17-Pad9)
Routing:
- net (no net): track 0.00 -> 1176.6 mm, vias 0 -> 4
- net unconnected-(U17-Pad9): track 0.00 -> 286.0 mm, vias 0 -> 3
- net +3.3VADC: track 280.1 -> 0.00 mm
- net +3V3: track 250.0 -> 0.00 mm, vias 3 -> 0
- net +3.3V-Switched: track 0.00 -> 173.9 mm, vias 0 -> 3
- net /MUX_COMMON: track 163.7 -> 0.00 mm, vias 2 -> 0
- net /SPI_CLK: track 159.8 -> 0.00 mm, vias 4 -> 0
- net /LEDs/LED_ROW_8: track 154.5 -> 0.00 mm
- net /LEDs/LED_ROW_7: track 153.5 -> 0.00 mm
- net unconnected-(U17-Pad40): track 0.00 -> 153.1 mm, vias 0 -> 1
- net /LEDs/LED_ROW_6: track 152.2 -> 0.00 mm
- net /LEDs/LED_ROW_4: track 149.8 -> 0.00 mm
- net /LEDs/LED_ROW_5: track 149.3 -> 0.00 mm
- net /LEDs/LED_ROW_3: track 147.7 -> 0.00 mm
- net /Buttons/BC_0: track 146.0 -> 0.00 mm, vias 2 -> 0
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Other:
- board text added: "A"
- board text added: "B"
- board text added: "DMX"
- board text added: "G"
- board text removed: "+"
- board text removed: "-"
- board text removed: "0"
- board text removed: "1"
- board text removed: "10"
- board text removed: "11"
- board text removed: "12"
- board text removed: "13"
- board text removed: "14"
- board text removed: "15"
- board text removed: "16"
- board text removed: "17"
- board text removed: "18"
- board text removed: "19"
- board text removed: "2"
- board text removed: "20"
- board text removed: "21"
- board text removed: "22"
- board text removed: "23"
- board text removed: "24"
- board text removed: "25"
- board text removed: "26"
- board text removed: "27"
- board text removed: "28"
- board text removed: "29"
- board text removed: "3"
- board text removed: "30"
- board text removed: "31"
- board text removed: "32"
- board text removed: "33"
- board text removed: "34"
- board text removed: "35"
- board text removed: "36"
- board text removed: "37"
- board text removed: "38"
- board text removed: "39"
- board text removed: "4"
- board text removed: "40"
- board text removed: "41"
- board text removed: "42"
- board text removed: "43"
- board text removed: "44"
- board text removed: "45"
- board text removed: "46"
- board text removed: "47"
- board text removed: "48"
- board text removed: "49"
- board text removed: "5"
- board text removed: "50"
- board text removed: "51"
- board text removed: "52"
- board text removed: "53"
- board text removed: "54"
- board text removed: "55"
- board text removed: "56"
- board text removed: "57"
- board text removed: "58"
- board text removed: "59"
- board text removed: "6"
- board text removed: "60"
- board text removed: "61"
- board text removed: "62"
- board text removed: "63"
- board text removed: "7"
- board text removed: "8"
- board text removed: "9"
- board text removed: "C0"
- board text removed: "C1"
- board text removed: "C2"
- board text removed: "C3"
- board text removed: "C4"
- board text removed: "C5"
- board text removed: "C6"
- board text removed: "C7"
- board text removed: "I2C"
- board text removed: "IN"
- board text removed: "NC"
- board text removed: "OUT"
- board text removed: "R0-R7"
- board text removed: "R8-R15"
- board text removed: "RX"
- board text removed: "S"
- board text removed: "SCL"
- board text removed: "SDA"
- board text removed: "TOUCHSCREEN"
- board text removed: "TX"

Commit message: Finalised schematic and PCB for MOOD Motherboard
Parts:
- removed D130: Red, LED_SMD:LED_0805_2012Metric
- removed R2300: 1k, Resistor_SMD:R_0402_1005Metric
- added BR1: DB107-BP, UltraLibrarian:DB-1_MCC, F.Cu at (228.2, 47.5)
- added BR2: DB107-BP, UltraLibrarian:DB-1_MCC, F.Cu at (226.2, 52.6)
- added C1: 1nF, Capacitor_SMD:C_0402_1005Metric, F.Cu at (228.8, 56.5)
- added C11: 10nF, Capacitor_SMD:C_0402_1005Metric, B.Cu at (223.8, 39.8)
- added C12: 10nF, Capacitor_SMD:C_0402_1005Metric, B.Cu at (223.8, 36.0)
- added C13: 10nF, Capacitor_SMD:C_0402_1005Metric, B.Cu at (223.8, 32.0)
- added C14: 10nF, Capacitor_SMD:C_0402_1005Metric, B.Cu at (223.8, 28.3)
- added C15: 1nF, Capacitor_SMD:C_0402_1005Metric, B.Cu at (218.0, 36.0)
- added C16: 1nF, Capacitor_SMD:C_0402_1005Metric, B.Cu at (217.0, 34.3)
- added C2: 100nF, Capacitor_SMD:C_0402_1005Metric, F.Cu at (229.8, 56.5)
- added C3: 47μF/100V, Capacitor_SMD:C_0402_1005Metric, F.Cu at (251.5, 52.2)
- added C31: 0.1μF, Capacitor_SMD:C_0402_1005Metric, F.Cu at (252.8, 67.0)
- added C33: 0.1μF, Capacitor_SMD:C_0402_1005Metric, F.Cu at (204.2, 46.5)
- added C34: 1μF, Capacitor_SMD:C_0402_1005Metric, F.Cu at (251.2, 67.0)
- added C35: 1μF, Capacitor_SMD:C_0402_1005Metric, F.Cu at (205.5, 46.5)
- added C36: 4.7mF, Capacitor_SMD:C_0402_1005Metric, F.Cu at (200.2, 52.0)
- added C37: 0.1μF, Capacitor_SMD:C_0402_1005Metric, F.Cu at (212.8, 67.8)
- added C38: 0.68μF, Capacitor_SMD:C_0402_1005Metric, F.Cu at (196.1, 62.2)
- added C39: 1μF, Capacitor_SMD:C_0402_1005Metric, F.Cu at (211.5, 67.8)
- added C4: 100nF/100V, Capacitor_SMD:C_0402_1005Metric, F.Cu at (246.6, 53.9)
- added C46: 100n, Capacitor_SMD:C_0402_1005Metric, F.Cu at (124.0, 52.8)
- added C47: 100n, Capacitor_SMD:C_0402_1005Metric, F.Cu at (118.0, 53.2)
- added C48: 100n, Capacitor_SMD:C_0402_1005Metric, F.Cu at (98.2, 46.0)
- added C49: 4.7u, Capacitor_SMD:C_0402_1005Metric, F.Cu at (109.2, 53.0)
- added C5: 5.6nF, Capacitor_SMD:C_0402_1005Metric, F.Cu at (252.8, 61.1)
- added C51: 10u, Capacitor_SMD:C_0402_1005Metric, F.Cu at (105.2, 52.8)
- added C52: 4.7μF, Capacitor_SMD:C_0402_1005Metric, F.Cu at (199.2, 30.0)
- added C53: 0.1μF, Capacitor_SMD:C_0402_1005Metric, F.Cu at (198.0, 30.0)
- added C54: 18pF, Capacitor_SMD:C_0402_1005Metric, F.Cu at (187.5, 35.2)
- added C55: 16pF, Capacitor_SMD:C_0402_1005Metric, F.Cu at (190.5, 35.2)
- added C6: 0.1μF, Capacitor_SMD:C_0402_1005Metric, F.Cu at (259.9, 60.8)
- added C7: 2.2μ, Capacitor_SMD:C_0402_1005Metric, F.Cu at (252.8, 64.8)
- added C8: 1nF, Capacitor_SMD:C_0402_1005Metric, B.Cu at (219.0, 34.3)
- added C9: 10μF, Capacitor_SMD:C_0402_1005Metric, F.Cu at (260.4, 65.2)
- added D1: BAV99S, Package_TO_SOT_SMD:SOT-363_SC-70-6, F.Cu at (194.6, 48.6)
- added D2: 1N5400, Diode_THT:D_DO-201AD_P15.24mm_Horizontal, F.Cu at (218.2, 67.2)
- added D3: 1N5400, Diode_THT:D_DO-201AD_P15.24mm_Horizontal, F.Cu at (212.2, 63.4)
- added D4: SMF58A, Diode_SMD:D_SMF, F.Cu at (231.8, 57.0)
- added D5: LED, LED_SMD:LED_0805_2012Metric, F.Cu at (254.6, 49.8)
- added D6: SMF58A, Diode_SMD:D_SMF, F.Cu at (258.2, 48.5)
- added D7: LED, LED_SMD:LED_0805_2012Metric, F.Cu at (250.0, 54.9)
- added D9: LED_Dual_AKA, LED_SMD:LED-L1T2_LUMILEDS, F.Cu at (189.8, 63.2)
- added F1: 0ZCF0030FF2C, UltraLibrarian:0ZCF0030FF2C, F.Cu at (223.0, 58.5)
- added J1: Conn_02x10_Odd_Even, Connector_PinHeader_2.54mm:PinHeader_2x10_P2.54mm_Vertical, F.Cu at (184.8, 71.4)
- added J13: On/Off Button, Connector_PinHeader_2.54mm:PinHeader_2x01_P2.54mm_Vertical, F.Cu at (204.5, 57.0)
- added J14: Kill Override, Connector_PinHeader_2.54mm:PinHeader_2x01_P2.54mm_Vertical, F.Cu at (197.5, 66.5)
- added J3: RJ45_LED_Shielded, Connector_RJ:RJ45_BEL_SS74301-00x_Vertical, F.Cu at (246.7, 39.6)
- added J4: 48V Out, Connector_PinHeader_2.54mm:PinHeader_1x02_P2.54mm_Vertical, F.Cu at (255.0, 52.5)
- added JP1: Jumper_3_Bridged12, Connector_PinHeader_2.54mm:PinHeader_1x03_P2.54mm_Vertical, F.Cu at (240.0, 58.7)
- added JP2: Jumper_3_Bridged12, Connector_PinHeader_2.54mm:PinHeader_1x03_P2.54mm_Vertical, F.Cu at (195.0, 70.5)
- added L1: 4.7μH, Inductor_SMD:L_0201_0603Metric, F.Cu at (259.9, 62.5)
- added Q1: AO3400A, Package_TO_SOT_SMD:SOT-23, F.Cu at (199.2, 49.0)
- added Q2: AO3401A, Package_TO_SOT_SMD:SOT-23, F.Cu at (176.0, 46.0)
- added Q3: AO3401A, Package_TO_SOT_SMD:SOT-23, F.Cu at (193.1, 58.2)
- added R1: 470, Resistor_SMD:R_0402_1005Metric, F.Cu at (232.7, 29.1)
- added R10: 75, Resistor_SMD:R_0402_1005Metric, B.Cu at (214.5, 39.8)
- added R11: 75, Resistor_SMD:R_0402_1005Metric, B.Cu at (214.5, 35.8)
- added R12: 75, Resistor_SMD:R_0402_1005Metric, B.Cu at (214.5, 32.0)
- added R13: 75, Resistor_SMD:R_0402_1005Metric, B.Cu at (214.5, 28.3)
- added R14: 10k, Resistor_SMD:R_0402_1005Metric, F.Cu at (251.5, 49.8)
- added R15: 10k, Resistor_SMD:R_0402_1005Metric, F.Cu at (251.5, 51.0)
- added R16: 10k, Resistor_SMD:R_0402_1005Metric, F.Cu at (252.1, 56.4)
- added R17: 10k, Resistor_SMD:R_0402_1005Metric, F.Cu at (247.8, 56.4)
- added R18: 19.1k, Resistor_SMD:R_0402_1005Metric, F.Cu at (252.6, 63.4)
- added R2: 470, Resistor_SMD:R_0402_1005Metric, B.Cu at (243.2, 29.2)
- added R21: 75, Resistor_SMD:R_0402_1005Metric, B.Cu at (221.5, 39.8)
- added R22: 75, Resistor_SMD:R_0402_1005Metric, B.Cu at (221.5, 36.0)
- added R23: 75, Resistor_SMD:R_0402_1005Metric, B.Cu at (221.5, 32.0)
- added R24: 75, Resistor_SMD:R_0402_1005Metric, B.Cu at (221.5, 28.3)
- added R25: 196k, Resistor_SMD:R_0402_1005Metric, F.Cu at (259.1, 65.2)
- added R26: 43.2k, Resistor_SMD:R_0402_1005Metric, F.Cu at (256.2, 66.5)
- added R27: 270k, Resistor_SMD:R_0402_1005Metric, F.Cu at (207.2, 69.2)
- added R29: 100k, Resistor_SMD:R_0402_1005Metric, F.Cu at (192.0, 70.5)
- added R3: 130k, Resistor_SMD:R_0402_1005Metric, F.Cu at (191.6, 47.6)
- added R30: 150k, Resistor_SMD:R_0402_1005Metric, F.Cu at (187.8, 47.8)
- added R36: 150k, Resistor_SMD:R_0402_1005Metric, F.Cu at (196.0, 56.8)
- added R38: 1k, Resistor_SMD:R_0402_1005Metric, F.Cu at (188.5, 66.8)
- added R39: 1k, Resistor_SMD:R_0402_1005Metric, F.Cu at (190.2, 66.8)
- added R4: 130k, Resistor_SMD:R_0402_1005Metric, F.Cu at (195.3, 51.1)
- added R47: 470, Resistor_SMD:R_0402_1005Metric, F.Cu at (126.2, 51.2)
- added R48: 50k, Resistor_SMD:R_0402_1005Metric, F.Cu at (118.7, 43.8)
- added R49: 133, Resistor_SMD:R_0402_1005Metric, F.Cu at (95.2, 43.0)
- added R5: 5.6MΩ, Resistor_SMD:R_0402_1005Metric, F.Cu at (200.3, 54.0)
- added R52: 12.4KΩ/1%, Resistor_SMD:R_0402_1005Metric, F.Cu at (207.0, 35.5)
- added R53: 4.7k, Resistor_SMD:R_0402_1005Metric, F.Cu at (189.0, 38.2)
- added R54: 4.7k, Resistor_SMD:R_0402_1005Metric, F.Cu at (192.2, 42.5)
- added R55: 1MΩ, Resistor_SMD:R_0402_1005Metric, F.Cu at (188.0, 36.7)
- added R56: 0Ω, Resistor_SMD:R_0402_1005Metric, F.Cu at (190.0, 36.8)
- added R6: 1270, Resistor_SMD:R_0402_1005Metric, F.Cu at (241.2, 55.7)
- added R7: 63.4, Resistor_SMD:R_0402_1005Metric, F.Cu at (233.8, 55.7)
- added R8: 25k, Resistor_SMD:R_0402_1005Metric, F.Cu at (239.4, 49.1)
- added R9: 100, Resistor_SMD:R_0402_1005Metric, F.Cu at (251.5, 48.2)
- added T1: H6062NL, UltraLibrarian:H6062FNLT_PUL, F.Cu at (219.5, 35.3)
- added U1: LTC2955xTS8-2, Package_TO_SOT_SMD:TSOT-23-8, F.Cu at (198.8, 61.2)
- added U12: TXB0104PW, Package_SO:TSSOP-14_4.4x5mm_P0.65mm, F.Cu at (121.0, 48.8)
- added U16: W5500, Package_QFP:LQFP-48_7x7mm_P0.5mm, F.Cu at (199.8, 37.2)
- added U3: TPS2378, Package_SO:Texas_HSOP-8-1EP_3.9x4.9mm_P1.27mm_ThermalVias, F.Cu at (243.9, 50.4)
- added U4: MAX17503SATP+, UltraLibrarian:21-100172_T2044+4C_MXM, F.Cu at (256.5, 61.8)
- added Y2: 25MHz, Crystal:Crystal_SMD_2520-4Pin_2.5x2.0mm, F.Cu at (187.5, 32.8)
- R50: value 33 -> 220
- R51: value 10 -> 220; moved to B.Cu
- U13: value MAX485 -> MAX485E; footprint Package_SO:SO-8_3.9x4.9mm_P1.27mm -> Package_SO:SOIC-8_3.9x4.9mm_P1.27mm
- U9: value SPX3819M5 -> SPX3819M5-L-3-3
- moved R50 104.8 mm to (106.5, 43.5)
- moved J5 104.0 mm to (152.5, 53.5), turned to -90 degrees
- moved R51 97.6 mm to (124.2, 43.5), turned to -90 degrees
- moved J9 97.2 mm to (111.8, 38.4)
- moved U13 81.1 mm to (99.8, 42.8), turned to 180 degrees
- moved C20 74.8 mm to (167.4, 57.1)
- moved C23 74.8 mm to (168.4, 57.1)
- moved C27 74.8 mm to (162.3, 56.8)
- moved C28 74.8 mm to (166.3, 59.2)
- moved J10 74.8 mm to (168.6, 65.0)
- moved R31 74.8 mm to (167.3, 59.2)
- moved R34 74.8 mm to (170.9, 58.8)
- moved Y1 74.8 mm to (164.3, 57.6)
- moved C19 74.8 mm to (159.8, 50.2)
- moved C22 74.8 mm to (170.7, 46.2)
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- renumbered J7 to J6, J6 to J7
Connections:
- C42 pad 2: +3V3 -> +3.3V-Supply
- C44 pad 2: +5V -> VBUS
- C45 pad 2: +5V -> VBUS
- C50 pad 2: +5V -> +5V-Switched
- D133 pad 4: +5V -> VBUS
- J12 pad 1: (no net) -> GND1
- J12 pad 2: (no net) -> Net-(J12-Pad2)
- J12 pad 3: (no net) -> Net-(J12-Pad3)
- J6 pad 3: +3V3 -> +3.3V-Switched
- J6 pad 4: +3V3 -> +3.3V-Switched
- J7 pad 3: +5V -> +5V-Switched
- J7 pad 4: +5V -> +5V-Switched
- J8 pad A4/B9: +5V -> VBUS
- J8 pad B4/A9: +5V -> VBUS
- J9 pad 2: GND -> GND1
- J9 pad 6: unconnected-(J1-Pad6) -> (no net)
- J9 pad 7: unconnected-(J1-Pad7) -> (no net)
- J9 pad 8: unconnected-(J1-Pad8) -> (no net)
- J9 pad 9: unconnected-(J1-Pad9) -> (no net)
- R50 pad 2: +3V3 -> +5V-SerialOut
- R51 pad 2: /MIDI_TX -> Net-(R51-Pad2)
- U13 pad 1: (no net) -> unconnected-(U13-Pad1)
- U13 pad 2: (no net) -> +5V-SerialOut
- U13 pad 3: (no net) -> +5V-SerialOut
- U13 pad 4: (no net) -> Net-(U12-Pad13)
- U13 pad 5: (no net) -> GND1
- U13 pad 6: (no net) -> Net-(J12-Pad3)
- U13 pad 7: (no net) -> Net-(J12-Pad2)
- U13 pad 8: (no net) -> +5V-SerialOut
- U14 pad 2: +5V -> +5V-Switched
- U14 pad 3: (no net) -> GND1
- U14 pad 4: (no net) -> +5V-SerialOut
- U15 pad 8: +3V3 -> +3.3V-Switched
- U17 pad 31: /SPI0_CS1 -> /SPI0_INT0
- U17 pad 32: /SPI0_CS2 -> /SPI0_CS1
- U17 pad 34: /SPI0_CS3 -> /SPI0_INT1
- U17 pad 35: /SPI0_CS4 -> /SPI0_CS2
- U17 pad 36: /SPI0_CS5 -> /SPI0_INT2
- U17 pad 37: /CLOCK_SUB -> /SPI0_CS3
- U17 pad 38: unconnected-(U17-Pad38) -> /SPI0_INT3
- U17 pad 39: unconnected-(U17-Pad39) -> /SPI0_CS4
- U17 pad 40: unconnected-(U17-Pad40) -> /SPI0_INT4
- U17 pad 41: unconnected-(U17-Pad41) -> /SPI0_CS5
- U17 pad 5: unconnected-(U17-Pad5) -> /CLOCK_SUB
- U17 pad 6: /DMI_TX -> /DMX_TX
- U17 pad 9: unconnected-(U17-Pad9) -> /SPI0_INT5
- U9 pad 1: +5V -> +5V-Supply
- U9 pad 3: +5V -> +5V-Supply
- U9 pad 5: +3V3 -> +3.3V-Supply
Routing:
- net (no net): track 1176.6 -> 0.00 mm, vias 4 -> 0
- net unconnected-(U17-Pad9): track 286.0 -> 0.00 mm, vias 3 -> 0
- net +5V: track 250.7 -> 0.00 mm, vias 1 -> 0
- net unconnected-(U17-Pad40): track 153.1 -> 0.00 mm, vias 1 -> 0
- net +3.3V-Supply: track 0.00 -> 145.8 mm, vias 0 -> 2
- net +5V-Switched: track 0.00 -> 138.2 mm, vias 0 -> 2
- net Net-(U11-Pad6): track 113.7 -> 0.00 mm
- net Net-(U11-Pad3): track 113.5 -> 0.00 mm
- net +5V-Supply: track 0.00 -> 109.0 mm, vias 0 -> 1
- net /Analog/MUX_S0_5V: track 103.4 -> 0.00 mm
- net /Analog/MUX_S1_5V: track 101.7 -> 0.00 mm
- net /Analog/MUX_S2_5V: track 91.2 -> 0.00 mm
- net /Analog/MUX_S3_5V: track 90.6 -> 0.00 mm
- net /PoE/+48VDC: track 0.00 -> 74.5 mm
- net /ETH_INTn: track 0.00 -> 73.2 mm, vias 0 -> 4
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- added copper zone on F.Cu, net /PoE/LX
- added copper zone on B.Cu, net EPAD
- added copper zone on F.Cu, net EPAD
Other:
- board size 181 x 97 mm -> 181 x 48.5 mm
- board text added: "MOOD Motherboard Revision: 0.1.1 2023.03"
- board text added: "https://shanteacontrols.com & Wayland Electronics"
- board text removed: "BTLDR"
- board text removed: "OpenDeck board Revision: 3.1.1 2022.11"
- board text removed: "PWR"
- board text removed: "https://shanteacontrols.com"
