File: bin/sch/MOOD/v0.1.1/Motherboard/MOOD-Motherboard-r0.1.1.kicad_sch (KiCad schematic)
At the start: 30 parts, among them J10 Conn_01x03, J11 Conn_01x02, J5 Conn_01x02, U15 W25Q128JVS, U17 RP2040, Y1 12MHz

Commit message: -	Made a bunch of changes -	Added KeyboardCard
Parts:
- removed U15: W25Q128JVS, Package_SO:SOIC-8_5.23x5.23mm_P1.27mm, symbol Igor:W25Q128JVS
- added U15: W25Q128JVS, Package_SO:SOIC-8_5.23x5.23mm_P1.27mm, symbol Memory_Flash:W25Q128JVS
- J1: renamed from J?; symbol Connector_Generic:Conn_02x10_Odd_Even -> Connector_Generic:Conn_02x08_Odd_Even
- gave numbers to parts that had none: 2
Connections:
- net +3V3 is gone; now on net +3.3V-Switched: R34.1, R35.1
- net QSPI__IO0 is gone; now on net SPI0_SCK: J1.5 (Pin_5)
- net +3.3V-Switched: now also J1.11 (Pin_11), U15.8 (VCC); no longer J1.15 (Pin_15)
- net +5V-Switched: now also J1.13 (Pin_13); no longer J1.17 (Pin_17)
- net GND: now also J1.15 (Pin_15), U15.4 (GND); no longer J1.19 (Pin_19)
- net QSPI_CLK: now also U15.6 (CLK); no longer J1.3 (Pin_3)
- net QSPI_CS: now also U15.1 (~{CS}); no longer J1.1 (Pin_1)
- net QSPI_IO0: now also U15.5 (DI(IO0))
- net QSPI_IO1: now also U15.2 (DO(IO1)); no longer J1.7 (Pin_7)
- net QSPI_IO2: now also U15.3 (IO2); no longer J1.9 (Pin_9)
- net QSPI_IO3: now also U15.7 (IO3); no longer J1.11 (Pin_11)
- net SPI0_CS0: now also J1.3 (Pin_3); no longer J1.4 (Pin_4)
- net SPI0_CS1: now also J1.2 (Pin_2); no longer J1.10 (Pin_10)
- net SPI0_CS2: now also J1.4 (Pin_4); no longer J1.12 (Pin_12)
- net SPI0_CS3: now also J1.6 (Pin_6); no longer J1.14 (Pin_14)
- net SPI0_CS4: now also J1.8 (Pin_8)
- net SPI0_RX: now also J1.1 (Pin_1); no longer J1.2 (Pin_2)
- net SPI0_SCK: no longer J1.6 (Pin_6)
- net SPI0_TX: now also J1.7 (Pin_7); no longer J1.8 (Pin_8)
- no-connect marks 4 -> 25
Other:
- sheet Ethernet_to_SPI ports: added none; removed ES_+3.3V, ES_GND
- sheet PoE ports: added DUPLEX_LED_C, ETH_MIDI_IN_LED_C, ETH_MIDI_OUT_LED_C; removed none
- sheet PowerSwitching ports: added none; removed GND, Supply-+3.3V , Switched-+3.3V , Switched-5VDC
- sheet USB ports: added none; removed USB_GND
- moved on the sheet: C17, C18, C19, C20, C21, C22, C23, C24, C25, C26, C27, C28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

Commit message: Redid power switching
Other:
- sheet PowerSwitching ports: added PSW_INT, PSW_KILL; removed none

Commit message: -	Hopefully finished schematics -	Started desining PCB for motherboard
Parts:
- removed U1, U2: 74HC595, symbol 74xx:74HC595
Connections:
- net INTn: no longer U17.16 (GPIO13)
- net SPI0_CS0: now also J1.2 (Pin_2); no longer J1.3 (Pin_3)
- net SPI0_CS1: now also J1.6 (Pin_6); no longer J1.2 (Pin_2)
- net SPI0_CS2: now also J1.10 (Pin_10); no longer J1.4 (Pin_4)
- net SPI0_CS3: now also J1.14 (Pin_14); no longer J1.6 (Pin_6)
- net SPI0_CS4: no longer J1.8 (Pin_8)
- net SPI0_TX: now also J1.3 (Pin_3); no longer J1.7 (Pin_7)
- net PSW_KILL: now reaches U17.17 (GPIO14)
- net PSW_INT: now reaches U17.18 (GPIO15)
- net CLOCK_SUB: now reaches U17.37 (GPIO25)
- net CLOCK_SUB: now also J1.9 (Pin_9)
- net SPI_INT2: now reaches J1.12 (Pin_12)
- net SPI_INT3: now reaches J1.16 (Pin_16)
- net LAL_CLOCK: no longer names the net of U17.8 (GPIO6)
- net LAL_DATA: no longer names the net of U17.7 (GPIO5)
- net LAL_LATCH: no longer names the net of U17.9 (GPIO7)
- net RSTn renamed ETH_RSTn
- new net ETH_INTn: U17.16 (GPIO13)
- new net SPI_INT0: J1.4 (Pin_4)
- new net SPI_INT1: J1.8 (Pin_8)
- no-connect marks 25 -> 14
Other:
- sheet DIN Serial ports: added none; removed DMX_TRAFFIC_OUT, MIDI_TRAFFIC_IN, MIDI_TRAFFIC_OUT
- sheet PoE ports: added none; removed DUPLEX_LED_A, DUPLEX_LED_C, ETH_MIDI_IN_LED_A, ETH_MIDI_IN_LED_C, ETH_MIDI_OUT_LED_A, ETH_MIDI_OUT_LED_C
- sheet USB ports: added none; removed USB_MIDI_TRAFFIC_IN, USB_MIDI_TRAFFIC_OUT
- note removed: "GPIO: LALs"
- note removed: "LAL: Link/Activity LEDs"
- note removed: "MLAL: MIDI Link/Activity LEDs (High = Link; send low for activity) MAL: MIDI Activity LEDs (Low = Default; send high for activity)"

Commit message: Finalised schematic and PCB for MOOD Motherboard
Parts:
- J1: footprint (none) -> Connector_PinHeader_2.54mm:PinHeader_2x10_P2.54mm_Vertical; symbol Connector_Generic:Conn_02x08_Odd_Even -> Connector_Generic:Conn_02x10_Odd_Even
Connections:
- net DMI_TX is gone; now on net DMX_TX: U17.6 (GPIO4)
- net SPI_INT3 is gone; now on net SPI0_INT3: J1.16 (Pin_16)
- net CLOCK_SUB: now also U17.5 (GPIO3); no longer U17.37 (GPIO25)
- net SPI0_CS1: now also U17.32 (GPIO21); no longer U17.31 (GPIO20)
- net SPI0_CS2: now also U17.35 (GPIO23); no longer U17.32 (GPIO21)
- net SPI0_CS3: now also U17.37 (GPIO25); no longer U17.34 (GPIO22)
- net SPI0_CS4: now also J1.18 (Pin_18), U17.39 (GPIO27_ADC1); no longer U17.35 (GPIO23)
- net SPI0_CS5: now also J1.19 (Pin_19), U17.41 (GPIO29_ADC3); no longer U17.36 (GPIO24)
- net SPI0_INT3: now reaches U17.38 (GPIO26_ADC0)
- net SPI0_INT4: now reaches U17.40 (GPIO28_ADC2)
- net SPI0_INT4: now also J1.20 (Pin_20)
- net SPI0_INT5: now reaches U17.9 (GPIO7)
- net SPI0_INT5: now also J1.17 (Pin_17)
- net SPI_INT0 renamed SPI0_INT0
- net SPI0_INT0: now also U17.31 (GPIO20)
- net SPI_INT1 renamed SPI0_INT1
- net SPI0_INT1: now also U17.34 (GPIO22)
- net SPI_INT2 renamed SPI0_INT2
- net SPI0_INT2: now also U17.36 (GPIO24)
- no-connect marks 14 -> 8
