File: bin/sch/MOOD/v0.1.1/Motherboard/PoE.kicad_sch (KiCad schematic)
At the start: 56 parts

Commit message: -	Made a bunch of changes -	Added KeyboardCard
Parts:
- C1, C11, C12, C13, C14, C15, C16, C2, C5, C6, C7, C8, C9: renamed from C?; footprint (none) -> Capacitor_SMD:C_0402_1005Metric
- D1: renamed from D?; value Green -> Blue
- D3: renamed from D?; value Blue -> Green
- T1: renamed from T?; symbol 2023-01-09_06-38-29:H6062FNLT -> UltraLibrarian:H6062FNLT
- U3: renamed from U?; symbol ModularDeck_Library:TPS2378 -> MOOD_Library:TPS2378
- gave numbers to parts that had none: 39
Connections:
- net GND: no longer D1.1 (K), D2.1 (K)
- net +3.3V renamed DUPLEX_LED_C
- new net ETH_MIDI_IN_LED_C: D1.1 (K)
- new net ETH_MIDI_OUT_LED_C: D2.1 (K)
Other:
- moved on the sheet: D1, D2, D3, J3, R1, R10, R11, R12, R13, R2, R3, R4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

Commit message: -	Hopefully finished schematics -	Started desining PCB for motherboard
Parts:
- removed D1, D2: Blue, LED_SMD:LED_0805_2012Metric, symbol Device:LED
- removed D3: Green, LED_SMD:LED_0805_2012Metric, symbol Device:LED
- removed R3: 680, Resistor_SMD:R_0402_1005Metric, symbol Device:R
- removed R4, R5: 1k, Resistor_SMD:R_0402_1005Metric, symbol Device:R
Changed lines of the file:
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@@
     (effects (font (size 1.27 1.27)) (justify left))
-  )
-  (hierarchical_label "DUPLEX_LED_A" (shape input) (at 34.29 78.74 180)
-    (effects (font (size 1.27 1.27)) (justify right))
   )
   (hierarchical_label "ETH_6_RX-" (shape input) (at 149.86 29.21 0)
     (effects (font (size 1.27 1.27)) (justify left))
   )
-  (hierarchical_label "ETH_MIDI_OUT_LED_A" (shape input) (at 34.29 71.12 180)
-    (effects (font (size 1.27 1.27)) (justify right))
-  )
   (hierarchical_label "ETH_4" (shape input) (at 149.86 36.83 0)
     (effects (font (size 1.27 1.27)) (justify left))
-  )
-  (hierarchical_label "ETH_MIDI_IN_LED_A" (shape input) (at 34.29 64.77 180)
-    (effects (font (size 1.27 1.27)) (justify right))
   )
   (hierarchical_label "GND" (shape output) (at 266.7 58.42 0)
@@
     (effects (font (size 1.27 1.27)) (justify right))
   )
-  (hierarchical_label "ETH_MIDI_IN_LED_C" (shape input) (at 49.53 64.77 0)
-    (effects (font (size 1.27 1.27)) (justify left))
-  )
   (hierarchical_label "GLED_C" (shape input) (at 20.32 25.4 180)
     (effects (font (size 1.27 1.27)) (justify right))
@@
     (effects (font (size 1.27 1.27)) (justify left))
   )
-  (hierarchical_label "DUPLEX_LED_C" (shape input) (at 49.53 78.74 0)
-    (effects (font (size 1.27 1.27)) (justify left))
-  )
   (hierarchical_label "YLED_A" (shape input) (at 20.32 43.18 180)
     (effects (font (size 1.27 1.27)) (justify right))
@@
   )
   (hierarchical_label "ETH_1_TX+" (shape input) (at 149.86 46.99 0)
-    (effects (font (size 1.27 1.27)) (justify left))
-  )
-  (hierarchical_label "ETH_MIDI_OUT_LED_C" (shape input) (at 49.53 71.12 0)
     (effects (font (size 1.27 1.27)) (justify left))
   )
@@
     (pin "2")
   )
-  (symbol (lib_id "Device:R") (at 38.1 64.77 90) (mirror x) (unit 1)
-    (in_bom yes) (on_board yes)
-    (property "Reference" "R3" (id 0) (at 38.1 67.31 90))
-    (property "Value" "680" (id 1) (at 38.1 64.77 90))
-    (property "Footprint" "Resistor_SMD:R_0402_1005Metric" (id 2) (at 38.1 62.992 90)
-      (effects (font (size 1.27 1.27)) hide)
-    )
-    (property "Datasheet" "~" (id 3) (at 38.1 64.77 0)
-      (effects (font (size 1.27 1.27)) hide)
-    )
-    (property "LCSC" "C25130" (id 4) (at 38.1 64.77 0)
-      (effects (font (size 1.27 1.27)) hide)
-    )
-    (pin "1")
-    (pin "2")
-  )
   (symbol (lib_id "Diode:SMF58A") (at 156.21 140.97 270) (unit 1)
     (in_bom yes) (on_board yes)
@@
     (pin "2")
   )
-  (symbol (lib_id "Device:R") (at 38.1 71.12 90) (mirror x) (unit 1)
-    (in_bom yes) (on_board yes)
-    (property "Reference" "R4" (id 0) (at 38.1 73.66 90))
-    (property "Value" "1k" (id 1) (at 38.1 71.12 90))
-    (property "Footprint" "Resistor_SMD:R_0402_1005Metric" (id 2) (at 38.1 69.342 90)
-      (effects (font (size 1.27 1.27)) hide)
-    )
-    (property "Datasheet" "~" (id 3) (at 38.1 71.12 0)
-      (effects (font (size 1.27 1.27)) hide)
-    )
-    (property "LCSC" "C11702" (id 4) (at 38.1 71.12 0)
-      (effects (font (size 1.27 1.27)) hide)
-    )
-    (pin "1")
-    (pin "2")
-  )
   (symbol (lib_id "Diode:SMF58A") (at 77.47 140.97 270) (unit 1)
     (in_bom yes) (on_board yes)
@@
     )
     (property "Datasheet" "~" (id 3) (at 166.37 50.8 0)
-      (effects (font (size 1.27 1.27)) hide)
-    )
-    (pin "1")
-    (pin "2")
-  )
-  (symbol (lib_id "Device:R") (at 38.1 78.74 90) (mirror x) (unit 1)
-    (in_bom yes) (on_board yes)
-    (property "Reference" "R5" (id 0) (at 38.1 81.28 90))
-    (property "Value" "1k" (id 1) (at 38.1 78.74 90))
-    (property "Footprint" "Resistor_SMD:R_0402_1005Metric" (id 2) (at 38.1 76.962 90)
-      (effects (font (size 1.27 1.27)) hide)
-    )
-    (property "Datasheet" "~" (id 3) (at 38.1 78.74 0)
-      (effects (font (size 1.27 1.27)) hide)
-    )
-    (property "LCSC" "C11702" (id 4) (at 38.1 78.74 0)
       (effects (font (size 1.27 1.27)) hide)
     )
@@
     (pin "2")
   )
-  (symbol (lib_id "Device:LED") (at 45.72 64.77 0) (mirror y) (unit 1)
-    (in_bom yes) (on_board yes)
-    (property "Reference" "D1" (id 0) (at 45.72 67.31 0))
-    (property "Value" "Blue" (id 1) (at 47.3075 69.85 0)
-      (effects (font (size 1.27 1.27)) hide)
-    )
-    (property "Footprint" "LED_SMD:LED_0805_2012Metric" (id 2) (at 45.72 64.77 0)
-      (effects (font (size 1.27 1.27)) hide)
-    )
-    (property "Datasheet" "~" (id 3) (at 45.72 64.77 0)
-      (effects (font (size 1.27 1.27)) hide)
-    )
-    (property "LCSC" "C142303" (id 4) (at 45.72 64.77 0)
-      (effects (font (size 1.27 1.27)) hide)
-    )
-    (pin "1")
-    (pin "2")
-  )
   (symbol (lib_id "power:GND") (at 191.77 165.1 0) (unit 1)
     (in_bom yes) (on_board yes) (fields_autoplaced)
@@
     (pin "2")
   )
-  (symbol (lib_id "Device:LED") (at 45.72 71.12 0) (mirror y) (unit 1)
-    (in_bom yes) (on_board yes)
-    (property "Reference" "D2" (id 0) (at 45.72 73.66 0))
-    (property "Value" "Blue" (id 1) (at 47.3075 76.2 0)
-      (effects (font (size 1.27 1.27)) hide)
-    )
-    (property "Footprint" "LED_SMD:LED_0805_2012Metric" (id 2) (at 45.72 71.12 0)
-      (effects (font (size 1.27 1.27)) hide)
-    )
-    (property "Datasheet" "~" (id 3) (at 45.72 71.12 0)
-      (effects (font (size 1.27 1.27)) hide)
-    )
-    (property "LCSC" "C84259" (id 4) (at 45.72 71.12 0)
-      (effects (font (size 1.27 1.27)) hide)
-    )
-    (pin "1")
-    (pin "2")
-  )
   (symbol (lib_id "Device:C") (at 255.27 123.19 90) (unit 1)
     (in_bom yes) (on_board yes) (fields_autoplaced)
@@
     (pin "4")
   )
-  (symbol (lib_id "Device:LED") (at 45.72 78.74 0) (mirror y) (unit 1)
-    (in_bom yes) (on_board yes)
-    (property "Reference" "D3" (id 0) (at 45.72 81.28 0))
-    (property "Value" "Green" (id 1) (at 47.3075 83.82 0)
-      (effects (font (size 1.27 1.27)) hide)
-    )
-    (property "Footprint" "LED_SMD:LED_0805_2012Metric" (id 2) (at 45.72 78.74 0)
-      (effects (font (size 1.27 1.27)) hide)
-    )
-    (property "Datasheet" "~" (id 3) (at 45.72 78.74 0)
-      (effects (font (size 1.27 1.27)) hide)
-    )
-    (property "LCSC" "C84259" (id 4) (at 45.72 78.74 0)
-      (effects (font (size 1.27 1.27)) hide)
-    )
-    (pin "1")
-    (pin "2")
-  )
   (symbol (lib_id "Device:R") (at 262.89 53.34 0) (unit 1)

Commit message: Finalised schematic and PCB for MOOD Motherboard
Parts:
- removed F1: Polyfuse, symbol Device:Polyfuse
- removed JP1: Jumper_3_Open, symbol Jumper:Jumper_3_Open
- added F1: 0ZCF0030FF2C, UltraLibrarian:0ZCF0030FF2C, symbol UltraLibrarian:0ZCF0030FF2C
- added JP1: Jumper_3_Bridged12, Connector_PinHeader_2.54mm:PinHeader_1x03_P2.54mm_Vertical, symbol Jumper:Jumper_3_Bridged12
- BR1, BR2: footprint DB-1_MCC -> UltraLibrarian:DB-1_MCC
- C3, C4: footprint (none) -> Capacitor_SMD:C_0402_1005Metric
- D5, D7: footprint (none) -> LED_SMD:LED_0805_2012Metric
- J3: footprint (none) -> Connector_RJ:RJ45_BEL_SS74301-00x_Vertical
- J4: value Conn_01x02_Male -> 48V Out; footprint (none) -> Connector_PinHeader_2.54mm:PinHeader_1x02_P2.54mm_Vertical
- L1: footprint (none) -> Inductor_SMD:L_0201_0603Metric
- R1, R10, R11, R12, R13, R14, R15, R16, R17, R18, R2, R21, R22, R23, R24, R25, R26, R6, R7, R8, R9: footprint (none) -> Resistor_SMD:R_0402_1005Metric
- T1: footprint H6062FNLT_PUL -> UltraLibrarian:H6062FNLT_PUL
- U4: footprint 21-100172_T2044+4C_MXM -> UltraLibrarian:21-100172_T2044+4C_MXM
Connections:
- net GND1 is gone; now on net GND: J3.SH
- net +48VDC: now also F1.2
- net GND: now also U4.21 (EPAD)
- net 2378-DEN: now reaches R8.2, U3.2 (DEN)
- net 2378-CLS: now reaches U3.3 (CLS)
- net 2378-CLS: now also JP1.2 (C)
- net EPAD: now reaches BR1.2 (-), BR2.2 (-), C1.2, C2.2, D4.2 (A2), R6.2, R7.2, U3.4 (VSS)
- net EPAD: now also U3.9 (EPAD)
- net 2378-CDB: now reaches R15.2, U3.6 (CDB)
- net 2378-T2P: now reaches R14.1, U3.7 (T2P)
- net 2378-APD: now reaches R9.1, U3.8 (APD)
- net at R7.1: now also JP1.3 (B)
- net Pre-Fuse-48V: now reaches BR1.1 (+), BR2.1 (+)
- net Pre-Fuse-48V: now also F1.1
- net BST: now reaches C6.1, U4.20 (BST)
- net LX: now reaches C6.2, L1.1, U4.17 (LX), U4.18 (LX), U4.19 (LX)
- net SS: now reaches C5.1, U4.7 (SS)
- net MX1+: now reaches J3.1, T1.23 (MX1+)
- net MX1-: now reaches J3.2, T1.22 (MX1-)
- net MX2+: now reaches J3.3, T1.20 (MX2+)
- net MX2-: now reaches J3.4, T1.19 (MX2-)
- net MX3+: now reaches J3.5, T1.17 (MX3+)
- net MX3-: now reaches J3.6, T1.16 (MX3-)
- net MX4+: now reaches J3.7, T1.14 (MX4+)
- net MX4-: now reaches J3.8, T1.13 (MX4-)
- net VCC: now reaches C7.2, U4.12 (VCC)
- net at R6.1: now also JP1.1 (A)
- net RT: now reaches R18.1, U4.10 (RT)
- no-connect marks 5 -> 4
Other:
- note added: "JP1: - Class 0 (1270Ω): 0.44-12.95W = 0.088-2.5A @ 5V - Class 4 (63.4Ω): 12.95-25.5W = 2.59-5.1A @ 5V"
