File: bin/sch/MOOD/v0.1.1/KeyboardCard/KeyboardCard-r3.1.0.kicad_sch (KiCad schematic)
At the start: 40 parts, among them J1 Conn_02x10_Odd_Even, J10 Conn_01x03, J11 Conn_01x02, J2 Conn_02x10_Odd_Even, J3 Conn_01x04, J4 Conn_01x03, J5 Conn_01x02, J6 Conn_01x04, J7 Conn_01x04, J8 Conn_01x04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

Commit message: -	Hopefully finished schematics -	Started desining PCB for motherboard
Parts:
- removed C17: 100n, Capacitor_SMD:C_0402_1005Metric, symbol Device:C
- removed C27, C28: 16p, Capacitor_SMD:C_0402_1005Metric, symbol Device:C
- removed J1, J2: Conn_02x10_Odd_Even, symbol Connector_Generic:Conn_02x10_Odd_Even
- removed J11: Conn_01x02, Connector_PinHeader_2.54mm:PinHeader_1x02_P2.54mm_Vertical, symbol Connector_Generic:Conn_01x02
- removed J4: Conn_01x03, symbol Connector_Generic:Conn_01x03
- removed R28, R31: 1k, Resistor_SMD:R_0402_1005Metric, symbol Device:R
- removed R32, R33: 27, Resistor_SMD:R_0402_1005Metric, symbol Device:R
- removed R35: 10k, Resistor_SMD:R_0402_1005Metric, symbol Device:R
- removed U15: W25Q128JVS, Package_SO:SOIC-8_5.23x5.23mm_P1.27mm, symbol Memory_Flash:W25Q128JVS
- removed Y1: 12MHz, Crystal:Crystal_SMD_2520-4Pin_2.5x2.0mm, symbol Igor:Crystal-4P
- added J1, J2: Conn_02x10_Odd_Even, symbol Connector_Generic:Conn_02x08_Odd_Even
- added J11, J4, J9: Conn_01x04, Connector_JST:JST_XH_B4B-XH-A_1x04_P2.50mm_Vertical, symbol Connector_Generic:Conn_01x04
- added U1: 74LVC1G32, symbol 74xGxx:74LVC1G32
Connections:
- net +3.3V: now also J1.11 (Pin_11), J11.1 (Pin_1), J11.2 (Pin_2), J11.3 (Pin_3), J11.4 (Pin_4), J2.11 (Pin_11), U1.5 (VCC); no longer R34.1
- net +5V: now also J1.13 (Pin_13), J2.13 (Pin_13)
- net GND: now also R34.1, J1.15 (Pin_15), J2.15 (Pin_15), J9.1 (Pin_1), J9.2 (Pin_2), J9.3 (Pin_3), J9.4 (Pin_4), U1.3 (GND)
- net SPI0_CS0: now also J1.2 (Pin_2), U1.1
- net SPI0_CS1: now also J1.6 (Pin_6), J2.2 (Pin_2)
- net SPI0_CS2: now also J1.10 (Pin_10), J2.6 (Pin_6)
- net SPI0_CS3: now also J1.14 (Pin_14), J2.10 (Pin_10)
- net SPI0_RX: now also J1.1 (Pin_1), J2.1 (Pin_1)
- net SPI0_SCK: now also J1.5 (Pin_5), J2.5 (Pin_5)
- net SPI0_TX: now also J1.3 (Pin_3), J2.3 (Pin_3)
- net at U17.38 (GPIO26_ADC0): now also J4.1 (Pin_1)
- net CLOCK_SUB: now reaches U17.20 (XIN)
- net CLOCK_SUB: now also J1.9 (Pin_9), J2.9 (Pin_9)
- net at R34.2, U17.26 (RUN): now also U1.2, U1.4
- net at U17.39 (GPIO27_ADC1): now also J4.2 (Pin_2)
- net at U17.40 (GPIO28_ADC2): now also J4.3 (Pin_3)
- net at U17.41 (GPIO29_ADC3): now also J4.4 (Pin_4)
- net QSPI_CLK: no longer names the net of U17.52 (QSPI_SCLK)
- net QSPI_CS: no longer names the net of U17.56 (QSPI_SS)
- net QSPI_IO0: no longer names the net of U17.53 (QSPI_SD0)
- net QSPI_IO1: no longer names the net of U17.55 (QSPI_SD1)
- net QSPI_IO2: no longer names the net of U17.54 (QSPI_SD2)
- net QSPI_IO3: no longer names the net of U17.51 (QSPI_SD3)
- new net SPI_INT0: J1.4 (Pin_4)
- new net SPI_INT1: J1.8 (Pin_8), J2.4 (Pin_4)
- new net SPI_INT2: J1.12 (Pin_12), J2.8 (Pin_8)
- new net SPI_INT3: J1.16 (Pin_16), J2.12 (Pin_12)
- no-connect marks 23 -> 25
Other:
- note added: "?GPIO: Button Columns"
- note added: "?SPI1: Button Rows"
- note added: "I2C"
- note added: "LED control"
- note added: "SPI0: Card Communication"
- note added: "UART: Touchscreen"
- moved on the sheet: R34
