File: bin/sch/MOOD/v0.1.1/KeyboardCard/Keypads.kicad_sch (KiCad schematic)
At the start: 42 parts, among them U4 TXB0104PW, U5 MAX7219, U6 74HC138, U8 74HC165

Commit message: -	Hopefully finished schematics -	Started desining PCB for motherboard
Parts:
- renumbered D3 to D10, D9 to D11, D4 to D12, D10 to D13, D5 to D2, D11 to D3, D6 to D4, D12 to D5, D7 to D6, D13 to D7, D2 to D8, D8 to D9
Changed lines of the file:
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@@
   (symbol (lib_id "Diode:1N4148WT") (at 231.14 38.1 0) (unit 1)
     (in_bom yes) (on_board yes)
-    (property "Reference" "D12" (id 0) (at 234.95 36.83 0))
+    (property "Reference" "D5" (id 0) (at 234.95 36.83 0))
     (property "Value" "~" (id 1) (at 231.14 34.29 0)
       (effects (font (size 1.27 1.27)) hide)
@@
   (symbol (lib_id "Diode:1N4148WT") (at 224.79 77.47 0) (unit 1)
     (in_bom yes) (on_board yes)
-    (property "Reference" "D3" (id 0) (at 233.68 76.2 0))
+    (property "Reference" "D10" (id 0) (at 233.68 76.2 0))
     (property "Value" "~" (id 1) (at 224.79 73.66 0)
       (effects (font (size 1.27 1.27)) hide)
@@
   (symbol (lib_id "Diode:1N4148WT") (at 231.14 33.02 0) (unit 1)
     (in_bom yes) (on_board yes)
-    (property "Reference" "D11" (id 0) (at 234.95 31.75 0))
+    (property "Reference" "D3" (id 0) (at 234.95 31.75 0))
     (property "Value" "~" (id 1) (at 231.14 29.21 0)
       (effects (font (size 1.27 1.27)) hide)
@@
   (symbol (lib_id "Diode:1N4148WT") (at 229.87 80.01 0) (unit 1)
     (in_bom yes) (on_board yes)
-    (property "Reference" "D9" (id 0) (at 233.68 78.74 0))
+    (property "Reference" "D11" (id 0) (at 233.68 78.74 0))
     (property "Value" "~" (id 1) (at 229.87 76.2 0)
       (effects (font (size 1.27 1.27)) hide)
@@
   (symbol (lib_id "Diode:1N4148WT") (at 226.06 35.56 0) (unit 1)
     (in_bom yes) (on_board yes)
-    (property "Reference" "D6" (id 0) (at 234.95 34.29 0))
+    (property "Reference" "D4" (id 0) (at 234.95 34.29 0))
     (property "Value" "~" (id 1) (at 226.06 31.75 0)
       (effects (font (size 1.27 1.27)) hide)
@@
   (symbol (lib_id "Diode:1N4148WT") (at 229.87 74.93 0) (unit 1)
     (in_bom yes) (on_board yes)
-    (property "Reference" "D8" (id 0) (at 233.68 73.66 0))
+    (property "Reference" "D9" (id 0) (at 233.68 73.66 0))
     (property "Value" "~" (id 1) (at 229.87 71.12 0)
       (effects (font (size 1.27 1.27)) hide)
@@
   (symbol (lib_id "Diode:1N4148WT") (at 224.79 72.39 0) (unit 1)
     (in_bom yes) (on_board yes)
-    (property "Reference" "D2" (id 0) (at 233.68 71.12 0))
+    (property "Reference" "D8" (id 0) (at 233.68 71.12 0))
     (property "Value" "~" (id 1) (at 224.79 68.58 0)
       (effects (font (size 1.27 1.27)) hide)
@@
   (symbol (lib_id "Diode:1N4148WT") (at 226.06 30.48 0) (unit 1)
     (in_bom yes) (on_board yes)
-    (property "Reference" "D5" (id 0) (at 234.95 29.21 0))
+    (property "Reference" "D2" (id 0) (at 234.95 29.21 0))
     (property "Value" "~" (id 1) (at 226.06 26.67 0)
       (effects (font (size 1.27 1.27)) hide)
@@
   (symbol (lib_id "Diode:1N4148WT") (at 226.06 40.64 0) (unit 1)
     (in_bom yes) (on_board yes)
-    (property "Reference" "D7" (id 0) (at 234.95 39.37 0))
+    (property "Reference" "D6" (id 0) (at 234.95 39.37 0))
     (property "Value" "~" (id 1) (at 226.06 36.83 0)
       (effects (font (size 1.27 1.27)) hide)
@@
   (symbol (lib_id "Diode:1N4148WT") (at 229.87 85.09 0) (unit 1)
     (in_bom yes) (on_board yes)
-    (property "Reference" "D10" (id 0) (at 233.68 83.82 0))
+    (property "Reference" "D13" (id 0) (at 233.68 83.82 0))
     (property "Value" "~" (id 1) (at 229.87 81.28 0)
       (effects (font (size 1.27 1.27)) hide)
@@
   (symbol (lib_id "Diode:1N4148WT") (at 231.14 43.18 0) (unit 1)
     (in_bom yes) (on_board yes)
-    (property "Reference" "D13" (id 0) (at 234.95 41.91 0))
+    (property "Reference" "D7" (id 0) (at 234.95 41.91 0))
     (property "Value" "~" (id 1) (at 231.14 39.37 0)
       (effects (font (size 1.27 1.27)) hide)
@@
   (symbol (lib_id "Diode:1N4148WT") (at 224.79 82.55 0) (unit 1)
     (in_bom yes) (on_board yes)
-    (property "Reference" "D4" (id 0) (at 233.68 81.28 0))
+    (property "Reference" "D12" (id 0) (at 233.68 81.28 0))
     (property "Value" "~" (id 1) (at 224.79 78.74 0)
       (effects (font (size 1.27 1.27)) hide)
